Commit message: update

File: data/models/basic/cube.urdf (robot description, URDF)
Before this commit: robot cuboid, 1 links, 0 joints
Links:
- link base_link: geometry collision mesh filename=obj/cube.obj scale=.01 .01 .01; visual mesh filename=obj/cube.obj scale=.01 .01 .01

File: data/models/basic/cylinder.urdf (robot description, URDF)
Before this commit: robot cube, 1 links, 0 joints
Links:
- link base_link: geometry collision mesh filename=obj/cylinder.obj scale=.01 .01 .01; visual mesh filename=obj/cylinder.obj scale=.01 .01 .01

File: data/models/basic/plus.urdf (robot description, URDF)
Before this commit: robot cuboid, 1 links, 0 joints
Links:
- link base_link: geometry collision mesh filename=obj/plus.obj scale=.01 .01 .01; visual mesh filename=obj/plus.obj scale=.01 .01 .01

File: data/models/basic/surface.urdf (robot description, URDF)
Before this commit: robot cube, 1 links, 0 joints
Links:
- link base_link: geometry collision box size=5.0 3.0 1; visual box size=4.1 1.8 1
